Commit message: gazebo tested

File: dji_description/urdf/dji_m100_gimbal_camera.xacro (robot description, xacro)
@@ -26,5 +26,5 @@
     parent_link="${namespace}/base_link"
     offset="0.05">
-    <origin xyz="0.0 0.0 0.0" rpy="0 0 0"/>
+    <origin xyz="0.0 0.0 -0.02" rpy="0 0 0"/>
   </xacro:gimbal_macro>
   <xacro:camera_macro
@@ -36,15 +36,15 @@
     camera_info_topic_name="camera_info"
     frame_rate="30"
-    horizontal_fov="0.72"
+    horizontal_fov="1.48"
     image_width="1280"
     image_height="1024"
     image_format="B8G8R8"
-    min_distance="0.1"
+    min_distance="0.72"
     max_distance="100"
     noise_mean="0.01"
-    noise_stddev="0.005"
+    noise_stddev="0.007"
     enable_visual="false"
-    k1="-0.0694"
-    k2="0.3306"
+    k1="0"
+    k2="0"
     k3="0"
     p1="0"
@@ -60,36 +60,4 @@
     <origin xyz="0.05 0 0" rpy="${pi/2} ${-pi/2} ${pi/2}" />
   </xacro:camera_macro>
-  <!-- <xacro:camera_macro
-    namespace="gimbal_camera"
-    parent_link="gimbal_camera/gimbal_link_2"
-    robot_namespace="/"
-    camera_name="camera"
-    image_topic_name="image_raw"
-    camera_info_topic_name="camera_info"
-    frame_rate="30"
-    horizontal_fov="0.73"
-    image_width="1280"
-    image_height="720"
-    image_format="B8G8R8"
-    min_distance="0.1"
-    max_distance="100"
-    noise_mean="0.01"
-    noise_stddev="0.005"
-    enable_visual="false"
-    k1="0.0"
-    k2="0.0"
-    k3="0.0"
-    p1="0.0"
-    p2="0.0"
-    cx="0.5"
-    cy="0.5">
-    <xacro:cylinder_inertial_with_origin
-      radius="0.01"
-      length="0.005"
-      mass="0.12">
-      <origin xyz="0 0 0" rpy="0 0 0" />
-    </xacro:cylinder_inertial_with_origin>
-    <origin xyz="0.05 0 0" rpy="${pi/2} ${-pi/2} ${-pi/2}" />
-  </xacro:camera_macro> -->
   <xacro:if value="$(arg is_kinematic)">
     <gazebo reference="${namespace}/base_link">
