Commit message: add simulator replay demo

File: dji_description/urdf/multirotor_base.xacro (robot description, xacro)
@@ -95,9 +95,9 @@
         </geometry>
       </visual>
-      <collision>
+      <!-- <collision>
         <geometry>
-          <cylinder length="0.005" radius="${radius_rotor}" /> <!-- [m] -->
+          <cylinder length="0.005" radius="${radius_rotor}" />
         </geometry>
-      </collision>
+      </collision> -->
     </link>
     <gazebo reference="${robot_namespace}/rotor_${motor_number}">
