Commit message: regular update

File: dji_description/urdf/dji_m100_default.xacro (robot description, xacro)
@@ -1,22 +1,39 @@
 <?xml version="1.0"?>
-<!--
-  Copyright 2015 Fadri Furrer, ASL, ETH Zurich, Switzerland
-  Copyright 2015 Michael Burri, ASL, ETH Zurich, Switzerland
-  Copyright 2015 Mina Kamel, ASL, ETH Zurich, Switzerland
-  Copyright 2015 Janosch Nikolic, ASL, ETH Zurich, Switzerland
-  Copyright 2015 Markus Achtelik, ASL, ETH Zurich, Switzerland
-  Licensed under the Apache License, Version 2.0 (the "License");
-  you may not use this file except in compliance with the License.
-  You may obtain a copy of the License at
-  http://www.apache.org/licenses/LICENSE-2.0
-  Unless required by applicable law or agreed to in writing, software
-  distributed under the License is distributed on an "AS IS" BASIS,
-  WITHOUT WARRANTIES OR CONDITIONS OF ANY KIND, either express or implied.
-  See the License for the specific language governing permissions and
-  limitations under the License.
--->
 <robot name="dji_m100" xmlns:xacro="http://ros.org/wiki/xacro">
   <xacro:arg name="is_kinematic" default="true"/>
   <xacro:include filename="$(find dji_description)/urdf/dji_m100.xacro" />
+  <xacro:include filename="$(find dji_description)/urdf/camera.xacro" />
+  <xacro:camera_macro
+    namespace="fixed_camera"
+    parent_link="${namespace}/base_link"
+    robot_namespace="/"
+    camera_name="camera"
+    image_topic_name="image_raw"
+    camera_info_topic_name="camera_info"
+    frame_rate="30"
+    horizontal_fov="1.48"
+    image_width="1280"
+    image_height="1024"
+    image_format="B8G8R8"
+    min_distance="0.72"
+    max_distance="100"
+    noise_mean="0.01"
+    noise_stddev="0.007"
+    enable_visual="false"
+    k1="0"
+    k2="0"
+    k3="0"
+    p1="0"
+    p2="0"
+    cx="0.5"
+    cy="0.5">
+    <xacro:cylinder_inertial_with_origin
+      radius="0.01"
+      length="0.005"
+      mass="0.12">
+      <origin xyz="0 0 0" rpy="0 0 0" />
+    </xacro:cylinder_inertial_with_origin>
+    <origin xyz="0 0.5 0" rpy="0 ${pi/2} ${-pi/2}" />
+  </xacro:camera_macro>
   <xacro:if value="$(arg is_kinematic)">
     <gazebo reference="${namespace}/base_link">

File: dji_description/urdf/dji_m100_gimbal_camera.xacro (robot description, xacro)
@@ -1,19 +1,3 @@
 <?xml version="1.0"?>
-<!--
-  Copyright 2015 Fadri Furrer, ASL, ETH Zurich, Switzerland
-  Copyright 2015 Michael Burri, ASL, ETH Zurich, Switzerland
-  Copyright 2015 Mina Kamel, ASL, ETH Zurich, Switzerland
-  Copyright 2015 Janosch Nikolic, ASL, ETH Zurich, Switzerland
-  Copyright 2015 Markus Achtelik, ASL, ETH Zurich, Switzerland
-  Licensed under the Apache License, Version 2.0 (the "License");
-  you may not use this file except in compliance with the License.
-  You may obtain a copy of the License at
-  http://www.apache.org/licenses/LICENSE-2.0
-  Unless required by applicable law or agreed to in writing, software
-  distributed under the License is distributed on an "AS IS" BASIS,
-  WITHOUT WARRANTIES OR CONDITIONS OF ANY KIND, either express or implied.
-  See the License for the specific language governing permissions and
-  limitations under the License.
--->
 <robot name="dji_m100" xmlns:xacro="http://ros.org/wiki/xacro">
   <xacro:include filename="$(find dji_description)/urdf/dji_m100.xacro" />
@@ -58,5 +42,5 @@
       <origin xyz="0 0 0" rpy="0 0 0" />
     </xacro:cylinder_inertial_with_origin>
-    <origin xyz="0.05 0 0" rpy="${pi/2} ${-pi/2} ${pi/2}" />
+    <origin xyz="0.05 0 0" rpy="${pi/2} ${-pi/2} 0" />
   </xacro:camera_macro>
   <xacro:if value="$(arg is_kinematic)">

File: dji_description/urdf/dji_m100_stereo_with_box.xacro (robot description, xacro)
@@ -1,19 +1,3 @@
 <?xml version="1.0"?>
-<!--
-  Copyright 2015 Fadri Furrer, ASL, ETH Zurich, Switzerland
-  Copyright 2015 Michael Burri, ASL, ETH Zurich, Switzerland
-  Copyright 2015 Mina Kamel, ASL, ETH Zurich, Switzerland
-  Copyright 2015 Janosch Nikolic, ASL, ETH Zurich, Switzerland
-  Copyright 2015 Markus Achtelik, ASL, ETH Zurich, Switzerland
-  Licensed under the Apache License, Version 2.0 (the "License");
-  you may not use this file except in compliance with the License.
-  You may obtain a copy of the License at
-  http://www.apache.org/licenses/LICENSE-2.0
-  Unless required by applicable law or agreed to in writing, software
-  distributed under the License is distributed on an "AS IS" BASIS,
-  WITHOUT WARRANTIES OR CONDITIONS OF ANY KIND, either express or implied.
-  See the License for the specific language governing permissions and
-  limitations under the License.
--->
 <robot name="dji_m100" xmlns:xacro="http://ros.org/wiki/xacro">
   <xacro:include filename="$(find dji_description)/urdf/dji_m100.xacro" />

File: dji_description/urdf/multirotor_base.xacro (robot description, xacro)
@@ -1,19 +1,3 @@
 <?xml version="1.0"?>
-<!--
-  Copyright 2015 Fadri Furrer, ASL, ETH Zurich, Switzerland
-  Copyright 2015 Michael Burri, ASL, ETH Zurich, Switzerland
-  Copyright 2015 Mina Kamel, ASL, ETH Zurich, Switzerland
-  Copyright 2015 Janosch Nikolic, ASL, ETH Zurich, Switzerland
-  Copyright 2015 Markus Achtelik, ASL, ETH Zurich, Switzerland
-  Licensed under the Apache License, Version 2.0 (the "License");
-  you may not use this file except in compliance with the License.
-  You may obtain a copy of the License at
-  http://www.apache.org/licenses/LICENSE-2.0
-  Unless required by applicable law or agreed to in writing, software
-  distributed under the License is distributed on an "AS IS" BASIS,
-  WITHOUT WARRANTIES OR CONDITIONS OF ANY KIND, either express or implied.
-  See the License for the specific language governing permissions and
-  limitations under the License.
--->
 <robot xmlns:xacro="http://ros.org/wiki/xacro">
   <!-- Macro for the inertia of a box -->

Commit message: add jing zhun chuan yue

File: dji_description/urdf/dji_m100_default.xacro (robot description, xacro)
@@ -3,37 +3,4 @@
   <xacro:arg name="is_kinematic" default="true"/>
   <xacro:include filename="$(find dji_description)/urdf/dji_m100.xacro" />
-  <xacro:include filename="$(find dji_description)/urdf/camera.xacro" />
-  <xacro:camera_macro
-    namespace="fixed_camera"
-    parent_link="${namespace}/base_link"
-    robot_namespace="/"
-    camera_name="camera"
-    image_topic_name="image_raw"
-    camera_info_topic_name="camera_info"
-    frame_rate="30"
-    horizontal_fov="1.48"
-    image_width="1280"
-    image_height="1024"
-    image_format="B8G8R8"
-    min_distance="0.72"
-    max_distance="100"
-    noise_mean="0.01"
-    noise_stddev="0.007"
-    enable_visual="false"
-    k1="0"
-    k2="0"
-    k3="0"
-    p1="0"
-    p2="0"
-    cx="0.5"
-    cy="0.5">
-    <xacro:cylinder_inertial_with_origin
-      radius="0.01"
-      length="0.005"
-      mass="0.12">
-      <origin xyz="0 0 0" rpy="0 0 0" />
-    </xacro:cylinder_inertial_with_origin>
-    <origin xyz="0 0.5 0" rpy="0 ${pi/2} ${-pi/2}" />
-  </xacro:camera_macro>
   <xacro:if value="$(arg is_kinematic)">
     <gazebo reference="${namespace}/base_link">
